File: electronics/eeZee_microSD.sch (EAGLE design)
At the start: 15 parts, among them U1 MCP1824S, U2 74HC4050

Commit message: Switched to push-pull socket, shrank board, modified regulator and level shifter layouts, modified silk layout.
Parts:
- removed C4: 10uF, rcl:CPOL-USSMCB
- removed U$1: MICROSD_TFLASH, mes_electromech:MICROSD_TFLASH
- added U3: USD-SOCKET, SparkFun-Connectors:USD-SOCKET
- C1: value 1uF -> 106; device rcl:C-USC0603 -> rcl:C-USC1206
- C2, C3: value 0.1uF -> 104
Connections:
- net !SS: now also U3.CS; no longer U$1.CS
- net GND: now also U3.CD1, U3.CD2, U3.GND, U3.SHIELD@1, U3.SHIELD@3; no longer C4.-, U$1.GND, U$1.SHIELD1, U$1.SHIELD2, U$1.SHIELD3, U$1.SHIELD4
- net MISO: now also U3.DO; no longer U$1.DO
- net MOSI: now also U3.DI; no longer U$1.DI
- net SCK: now also U3.SCK; no longer U$1.SCK
- net VBOARD: no longer C4.+
- net VCC: now also U3.VCC; no longer U$1.VCC
